Commit message: added realsense-ros

File: omniwheel_ros/src/omniwheel_visualization/src/description/omniwheel_description.urdf (robot description, URDF)
Before this commit: robot omniwheel, 2 links, 1 joints
Links:
- link base_link: geometry collision cylinder length=0.09 radius=0.175; visual cylinder length=0.09 radius=0.175

Commit message: Added lidar pointcloud2 topic

File: omniwheel_ros/src/omniwheel_visualization/src/description/omniwheel_description.urdf (robot description, URDF)
Before this commit: robot omniwheel, 2 links, 1 joints
Links:
- added link lidar_link, mass 0.125; collision cylinder length=0.025 radius=0.03; visual cylinder length=0.025 radius=0.03
Joints:
- added joint lidar_joint: type fixed, parent base_link, child lidar_link, origin xyz=0 0 0.07 rpy=-1.57 0 0

Commit message: Changed base_footprint tf

File: omniwheel_ros/src/omniwheel_visualization/src/description/omniwheel_description.urdf (robot description, URDF)
Before this commit: robot omniwheel, 3 links, 2 joints
Joints:
- joint base_joint: origin xyz=0.0 0.0 0.0 rpy=0 0 0 -> xyz=0.0 0.0 -0.065 rpy=0 0 0
- joint lidar_joint: origin xyz=0 0 0.07 rpy=-1.57 0 0 -> xyz=0 0 0.175 rpy=-1.57 0 0
